Commit message: .

File: robofin/urdf/franka_panda/panda.urdf (robot description, URDF)
Before this commit: robot panda, 14 links, 13 joints
Links:
- removed link right_gripper
- link panda_hand: geometry collision mesh filename=package://meshes/collision/hand.obj; visual mesh filename=package://meshes/visual/hand.obj
- link panda_leftfinger: geometry collision mesh filename=package://meshes/collision/finger.obj; visual mesh filename=package://meshes/visual/finger.obj
- link panda_link0: geometry collision mesh filename=package://meshes/collision/link0.obj; visual mesh filename=package://meshes/collision/link0.obj
- link panda_link1: geometry collision mesh filename=package://meshes/collision/link1.obj; visual mesh filename=package://meshes/visual/link1.obj
- link panda_link2: geometry collision mesh filename=package://meshes/collision/link2.obj; visual mesh filename=package://meshes/visual/link2.obj
- link panda_link3: geometry collision mesh filename=package://meshes/collision/link3.obj; visual mesh filename=package://meshes/visual/link3.obj
- link panda_link4: geometry collision mesh filename=package://meshes/collision/link4.obj; visual mesh filename=package://meshes/visual/link4.obj
- link panda_link5: geometry collision mesh filename=package://meshes/collision/link5.obj; visual mesh filename=package://meshes/visual/link5.obj
- link panda_link6: geometry collision mesh filename=package://meshes/collision/link6.obj; visual mesh filename=package://meshes/visual/link6.obj
- link panda_link7: geometry collision mesh filename=package://meshes/collision/link7.obj; visual mesh filename=package://meshes/collision/link7.obj
- link panda_rightfinger: geometry collision mesh filename=package://meshes/collision/finger.obj; visual mesh filename=package://meshes/visual/finger.obj
Joints:
- removed joint right_gripper
- joint panda_joint1: limit lower=-2.8973 upper=2.8973 effort=87 velocity=2.1750 -> lower=-2.9671 upper=2.9671 effort=87 velocity=2.1750
- joint panda_joint2: limit lower=-1.7628 upper=1.7628 effort=87 velocity=2.1750 -> lower=-1.8326 upper=1.8326 effort=87 velocity=2.1750
- joint panda_joint3: limit lower=-2.8973 upper=2.8973 effort=87 velocity=2.1750 -> lower=-2.9671 upper=2.9671 effort=87 velocity=2.1750
- joint panda_joint4: limit lower=-3.0718 upper=-0.0698 effort=87 velocity=2.1750 -> lower=-3.1416 upper=0.0 effort=87 velocity=2.1750
- joint panda_joint5: limit lower=-2.8973 upper=2.8973 effort=12 velocity=2.6100 -> lower=-2.9671 upper=2.9671 effort=12 velocity=2.6100
- joint panda_joint6: limit lower=-0.0175 upper=3.7525 effort=12 velocity=2.6100 -> lower=-0.0873 upper=3.8223 effort=12 velocity=2.6100
- joint panda_joint7: limit lower=-2.8973 upper=2.8973 effort=12 velocity=2.6100 -> lower=-2.9671 upper=2.9671 effort=12 velocity=2.6100
